Commit message: Added gps_link and imu_link to URDF
Signed-off-by: Alberto Tudela <ajtudela@gmail.com>

File: pioneer_description/urdf/pioneer3at.xacro (robot description, xacro)
@@ -17,14 +17,14 @@
 -->
 <robot name="Pioneer3AT"
-       xmlns:xacro="http://ros.org/wiki/xacro">
-       <!-- Calibration data -->
-       <xacro:include filename="pioneer3at_calibration.xacro" />
-       <!-- Robot body definition -->
-       <xacro:include filename="pioneer3at_body.xacro"/>
-       <!-- Instantiate front wheels -->
-       <xacro:p3at_front suffix="left" reflect="1"/>
-       <xacro:p3at_front suffix="right" reflect="-1"/>
-       <!-- Instantiate back wheels -->
-       <xacro:p3at_back suffix="left" reflect="1"/>
-       <xacro:p3at_back suffix="right" reflect="-1"/>
+  xmlns:xacro="http://ros.org/wiki/xacro">
+  <!-- Calibration data -->
+  <xacro:include filename="pioneer3at_calibration.xacro" />
+  <!-- Robot body definition -->
+  <xacro:include filename="pioneer3at_body.xacro"/>
+  <!-- Instantiate front wheels -->
+  <xacro:p3at_front suffix="left" reflect="1"/>
+  <xacro:p3at_front suffix="right" reflect="-1"/>
+  <!-- Instantiate back wheels -->
+  <xacro:p3at_back suffix="left" reflect="1"/>
+  <xacro:p3at_back suffix="right" reflect="-1"/>
 </robot>

File: pioneer_description/urdf/pioneer3at_body.xacro (robot description, xacro)
@@ -167,4 +167,44 @@
     <child link="back_sonar"/>
   </joint>
+  <!-- GPS -->
+  <link name="gps_link">
+    <inertial>
+      <mass value="0.05"/>
+      <origin xyz="0 0 0"/>
+      <inertia ixx="0.001" ixy="0.0" ixz="0.0" iyy="0.001" iyz="0.0" izz="0.001"/>
+    </inertial>
+    <visual name="gps_visual">
+      <origin xyz="0 0 0" rpy="0 0 0"/>
+      <geometry>
+        <box size="0.05 0.05 0.05"/>
+      </geometry>
+      <material name="white"/>
+    </visual>
+  </link>
+  <joint name="base_gps_joint" type="fixed">
+    <origin xyz="${gps_trans_x} ${gps_trans_y} ${gps_trans_z}" rpy="${gps_rot_x} ${gps_rot_y} ${gps_rot_z}"/>
+    <parent link="top_plate"/>
+    <child link="gps_link"/>
+  </joint>
+  <!-- IMU -->
+  <link name="imu_link">
+    <inertial>
+      <mass value="0.05"/>
+      <origin xyz="0 0 0"/>
+      <inertia ixx="0.001" ixy="0.0" ixz="0.0" iyy="0.001" iyz="0.0" izz="0.001"/>
+    </inertial>
+    <visual name="imu_visual">
+      <origin xyz="0 0 0" rpy="0 0 0"/>
+      <geometry>
+        <box size="0.04 0.04 0.04"/>
+      </geometry>
+      <material name="white"/>
+    </visual>
+  </link>
+  <joint name="base_imu_joint" type="fixed">
+    <origin xyz="${imu_trans_x} ${imu_trans_y} ${imu_trans_z}" rpy="${imu_rot_x} ${imu_rot_y} ${imu_rot_z}"/>
+    <parent link="top_plate"/>
+    <child link="imu_link"/>
+  </joint>
   <!-- Front Axles + Wheels + Hubcaps -->
   <xacro:macro name="p3at_front" params="suffix reflect">

File: pioneer_description/urdf/pioneer3at_calibration.xacro (robot description, xacro)
@@ -17,70 +17,84 @@
 -->
 <robot name="Pioneer3AT"
-    xmlns:xacro="http://ros.org/wiki/xacro">
-    <!-- Xacro properties -->
-    <xacro:property name="base_link_height" value="0.177" />
-    <!-- Calibration params -->
-    <!-- Footprint -->
-    <xacro:property name="footprint_trans_x" value="0.0" />
-    <xacro:property name="footprint_trans_y" value="0.0" />
-    <xacro:property name="footprint_trans_z" value="0.0" />
-    <xacro:property name="footprint_rot_x" value="0.0" />
-    <xacro:property name="footprint_rot_y" value="0.0" />
-    <xacro:property name="footprint_rot_z" value="0.0" />
-    <!-- Top laser (base_laser_link) -->
-    <xacro:property name="top_laser_trans_x" value="0.0" />
-    <xacro:property name="top_laser_trans_y" value="0.0" />
-    <xacro:property name="top_laser_trans_z" value="0.23" />
-    <xacro:property name="top_laser_rot_x" value="0.0" />
-    <xacro:property name="top_laser_rot_y" value="0.0" />
-    <xacro:property name="top_laser_rot_z" value="0.0" />
-    <!-- Intel RealSense D455 relative to the body frame -->
-    <xacro:property name="realsense_trans_x" value="0.225" />
-    <xacro:property name="realsense_trans_y" value="0.0" />
-    <xacro:property name="realsense_trans_z" value="0.45" />
-    <xacro:property name="realsense_rot_x" value="0.0" />
-    <xacro:property name="realsense_rot_y" value="0.0" />
-    <xacro:property name="realsense_rot_z" value="0.0" />
-    <!-- Front Sonar -->
-    <xacro:property name="front_sonar_trans_x" value="0.193" />
-    <xacro:property name="front_sonar_trans_y" value="0.0" />
-    <xacro:property name="front_sonar_trans_z" value="0.25" />
-    <xacro:property name="front_sonar_rot_x" value="0.0" />
-    <xacro:property name="front_sonar_rot_y" value="0.0" />
-    <xacro:property name="front_sonar_rot_z" value="0.0" />
-    <!-- Back Sonar -->
-    <xacro:property name="back_sonar_trans_x" value="-0.187" />
-    <xacro:property name="back_sonar_trans_y" value="0.0" />
-    <xacro:property name="back_sonar_trans_z" value="0.247" />
-    <xacro:property name="back_sonar_rot_x" value="0.0" />
-    <xacro:property name="back_sonar_rot_y" value="0.0" />
-    <xacro:property name="back_sonar_rot_z" value="0.0" />
-    <!-- Front Axles -->
-    <xacro:property name="front_left_axle_trans_x" value="0.135" />
-    <xacro:property name="front_left_axle_trans_y" value="0.156" />
-    <xacro:property name="front_left_axle_trans_z" value="0.111" />
-    <xacro:property name="front_right_axle_trans_x" value="0.135" />
-    <xacro:property name="front_right_axle_trans_y" value="-0.156" />
-    <xacro:property name="front_right_axle_trans_z" value="0.111" />
-    <!-- Back Axles -->
-    <xacro:property name="back_left_axle_trans_x" value="-0.134" />
-    <xacro:property name="back_left_axle_trans_y" value="0.156" />
-    <xacro:property name="back_left_axle_trans_z" value="0.111" />
-    <xacro:property name="back_right_axle_trans_x" value="-0.134" />
-    <xacro:property name="back_right_axle_trans_y" value="-0.156" />
-    <xacro:property name="back_right_axle_trans_z" value="0.111" />
-    <!-- Top Laser Support (lidar support) -->
-    <xacro:property name="top_laser_support_trans_x" value="-0.07" />
-    <xacro:property name="top_laser_support_trans_y" value="0.0" />
-    <xacro:property name="top_laser_support_trans_z" value="0.0" />
-    <xacro:property name="top_laser_support_rot_x" value="0.0" />
-    <xacro:property name="top_laser_support_rot_y" value="0.0" />
-    <xacro:property name="top_laser_support_rot_z" value="0.0" />
-    <!-- Top RealSense Support -->
-    <xacro:property name="top_realsense_trans_x" value="0.225" />
-    <xacro:property name="top_realsense_trans_y" value="0.0" />
-    <xacro:property name="top_realsense_trans_z" value="0.0" />
-    <xacro:property name="top_realsense_rot_x" value="0.0" />
-    <xacro:property name="top_realsense_rot_y" value="0.0" />
-    <xacro:property name="top_realsense_rot_z" value="0.0" />
+  xmlns:xacro="http://ros.org/wiki/xacro">
+  <!-- Xacro properties -->
+  <xacro:property name="base_link_height" value="0.177" />
+  <!-- Calibration params -->
+  <!-- Footprint -->
+  <xacro:property name="footprint_trans_x" value="0.0" />
+  <xacro:property name="footprint_trans_y" value="0.0" />
+  <xacro:property name="footprint_trans_z" value="0.0" />
+  <xacro:property name="footprint_rot_x" value="0.0" />
+  <xacro:property name="footprint_rot_y" value="0.0" />
+  <xacro:property name="footprint_rot_z" value="0.0" />
+  <!-- Top laser (base_laser_link) -->
+  <xacro:property name="top_laser_trans_x" value="0.0" />
+  <xacro:property name="top_laser_trans_y" value="0.0" />
+  <xacro:property name="top_laser_trans_z" value="0.23" />
+  <xacro:property name="top_laser_rot_x" value="0.0" />
+  <xacro:property name="top_laser_rot_y" value="0.0" />
+  <xacro:property name="top_laser_rot_z" value="0.0" />
+  <!-- Intel RealSense D455 relative to the body frame -->
+  <xacro:property name="realsense_trans_x" value="0.225" />
+  <xacro:property name="realsense_trans_y" value="0.0" />
+  <xacro:property name="realsense_trans_z" value="0.45" />
+  <xacro:property name="realsense_rot_x" value="0.0" />
+  <xacro:property name="realsense_rot_y" value="0.0" />
+  <xacro:property name="realsense_rot_z" value="0.0" />
+  <!-- Front Sonar -->
+  <xacro:property name="front_sonar_trans_x" value="0.193" />
+  <xacro:property name="front_sonar_trans_y" value="0.0" />
+  <xacro:property name="front_sonar_trans_z" value="0.25" />
+  <xacro:property name="front_sonar_rot_x" value="0.0" />
+  <xacro:property name="front_sonar_rot_y" value="0.0" />
+  <xacro:property name="front_sonar_rot_z" value="0.0" />
+  <!-- Back Sonar -->
+  <xacro:property name="back_sonar_trans_x" value="-0.187" />
+  <xacro:property name="back_sonar_trans_y" value="0.0" />
+  <xacro:property name="back_sonar_trans_z" value="0.247" />
+  <xacro:property name="back_sonar_rot_x" value="0.0" />
+  <xacro:property name="back_sonar_rot_y" value="0.0" />
+  <xacro:property name="back_sonar_rot_z" value="0.0" />
+  <!-- Front Axles -->
+  <xacro:property name="front_left_axle_trans_x" value="0.135" />
+  <xacro:property name="front_left_axle_trans_y" value="0.156" />
+  <xacro:property name="front_left_axle_trans_z" value="0.111" />
+  <xacro:property name="front_right_axle_trans_x" value="0.135" />
+  <xacro:property name="front_right_axle_trans_y" value="-0.156" />
+  <xacro:property name="front_right_axle_trans_z" value="0.111" />
+  <!-- Back Axles -->
+  <xacro:property name="back_left_axle_trans_x" value="-0.134" />
+  <xacro:property name="back_left_axle_trans_y" value="0.156" />
+  <xacro:property name="back_left_axle_trans_z" value="0.111" />
+  <xacro:property name="back_right_axle_trans_x" value="-0.134" />
+  <xacro:property name="back_right_axle_trans_y" value="-0.156" />
+  <xacro:property name="back_right_axle_trans_z" value="0.111" />
+  <!-- Top Laser Support (lidar support) -->
+  <xacro:property name="top_laser_support_trans_x" value="-0.07" />
+  <xacro:property name="top_laser_support_trans_y" value="0.0" />
+  <xacro:property name="top_laser_support_trans_z" value="0.0" />
+  <xacro:property name="top_laser_support_rot_x" value="0.0" />
+  <xacro:property name="top_laser_support_rot_y" value="0.0" />
+  <xacro:property name="top_laser_support_rot_z" value="0.0" />
+  <!-- Top RealSense Support -->
+  <xacro:property name="top_realsense_trans_x" value="0.225" />
+  <xacro:property name="top_realsense_trans_y" value="0.0" />
+  <xacro:property name="top_realsense_trans_z" value="0.0" />
+  <xacro:property name="top_realsense_rot_x" value="0.0" />
+  <xacro:property name="top_realsense_rot_y" value="0.0" />
+  <xacro:property name="top_realsense_rot_z" value="0.0" />
+  <!-- GPS -->
+  <xacro:property name="gps_trans_x" value="0.0" />
+  <xacro:property name="gps_trans_y" value="0.10" />
+  <xacro:property name="gps_trans_z" value="0.0" />
+  <xacro:property name="gps_rot_x" value="0.0" />
+  <xacro:property name="gps_rot_y" value="0.0" />
+  <xacro:property name="gps_rot_z" value="0.0" />
+  <!-- IMU -->
+  <xacro:property name="imu_trans_x" value="0.0" />
+  <xacro:property name="imu_trans_y" value="-0.10" />
+  <xacro:property name="imu_trans_z" value="0.0" />
+  <xacro:property name="imu_rot_x" value="0.0" />
+  <xacro:property name="imu_rot_y" value="0.0" />
+  <xacro:property name="imu_rot_z" value="0.0" />
 </robot>
